File: connector-breakout-a1/connector-breakout-a1.kicad_pcb (KiCad board)
At the start: 2 copper layers, 17.5 x 40 mm, 18 parts, among them J1 Ruuvi Connector Horizontal, J2 Ruuvi Connector Pin Header, J3 Ruuvi Connector Pin Header, J4 Ruuvi Connector Horizontal

Commit message: First draft
Parts:
- removed the G*** at (87.4, 91.0)
- removed the G*** at (87.4, 82.1)
- removed the G*** at (85.7, 101.7)
- removed the G*** at (95.6, 88.9)
- removed the G*** at (98.4, 101.7)
- removed the G*** at (96.6, 82.1)
- removed the G*** at (96.7, 91.0)
- removed the G*** at (92.1, 80.7)
- removed J1: Ruuvi Connector Horizontal, connector:RUUVI_CONNECTOR_FFC
- added C1: 100n, passives:CAPC160X80X35L25N, F.Cu at (95.0, 96.4)
- added G***: EYESILK2MM, ruuvi:EYESILK2MM, F.Cu at (91.0, 80.1)
- added JP1: SolderJumper_3_Open, Jumper:SolderJumper-3_P2.0mm_Open_TrianglePad1.0x1.5mm_NumberLabels, B.Cu at (92.0, 87.5)
- added JP2: SolderJumper_3_Open, Jumper:SolderJumper-3_P2.0mm_Open_TrianglePad1.0x1.5mm_NumberLabels, B.Cu at (92.0, 91.3)
- added JP3: SolderJumper_3_Open, Jumper:SolderJumper-3_P2.0mm_Open_TrianglePad1.0x1.5mm_NumberLabels, B.Cu at (92.0, 95.1)
- added R1: 10k, passives:CAPC160X80X35L25N, F.Cu at (94.0, 81.7)
- added R2: 10k, passives:CAPC160X80X35L25N, F.Cu at (95.6, 81.7)
- added U1: NPA-700, Package_SO:SOIC-14W_7.5x9mm_P1.27mm, F.Cu at (92.0, 89.3)
- moved J4 0.06 mm to (92.0, 100.5)
Connections:
- J2 pad 1: Net-(J2-Pad1) -> /VDD
- J2 pad 2: Net-(J2-Pad2) -> /SCL
- J2 pad 3: Net-(J2-Pad3) -> /SDA
- J2 pad 4: Net-(J2-Pad4) -> /GPIO3
- J2 pad 5: Net-(J2-Pad5) -> /GPIO4
- J2 pad 6: Net-(J2-Pad6) -> /GPIO5
- J2 pad 7: Net-(J2-Pad7) -> /GPIO6
- J2 pad 8: Net-(J2-Pad8) -> /GND
- J3 pad 1: Net-(J1-Pad1) -> /VDD
- J3 pad 2: Net-(J1-Pad2) -> /SCL
- J3 pad 3: Net-(J1-Pad3) -> /SDA
- J3 pad 4: Net-(J1-Pad4) -> /GPIO3
- J3 pad 5: Net-(J1-Pad5) -> /GPIO4
- J3 pad 6: Net-(J1-Pad6) -> /GPIO5
- J3 pad 7: Net-(J1-Pad7) -> /GPIO6
- J3 pad 8: Net-(J1-Pad8) -> /GND
- J4 pad 1: Net-(J2-Pad1) -> /VDD
- J4 pad 2: Net-(J2-Pad2) -> /SCL
- J4 pad 3: Net-(J2-Pad3) -> /SDA
- J4 pad 4: Net-(J2-Pad4) -> /GPIO3
- J4 pad 5: Net-(J2-Pad5) -> /GPIO4
- J4 pad 6: Net-(J2-Pad6) -> /GPIO5
- J4 pad 7: Net-(J2-Pad7) -> /GPIO6
- J4 pad 8: Net-(J2-Pad8) -> /GND
Routing:
- net /VDD: track 0.00 -> 58.8 mm, vias 0 -> 5
- net /SCL: track 0.00 -> 42.1 mm, vias 0 -> 2
- net /SDA: track 0.00 -> 42.0 mm, vias 0 -> 1
- net /GND: track 0.00 -> 38.1 mm, vias 0 -> 4
- net /GPIO4: track 0.00 -> 27.9 mm, vias 0 -> 3
- net /GPIO3: track 0.00 -> 24.0 mm, vias 0 -> 1
- net /GPIO6: track 0.00 -> 19.3 mm, vias 0 -> 2
- net /GPIO5: track 0.00 -> 17.1 mm, vias 0 -> 1
- removed copper zone on F.Cu, net (none)
- removed copper zone on B.Cu, net Net-(J1-Pad1)
- removed copper zone on B.Cu, net Net-(J1-Pad2)
- removed copper zone on B.Cu, net Net-(J1-Pad3)
- removed copper zone on B.Cu, net Net-(J1-Pad4)
- removed copper zone on B.Cu, net Net-(J1-Pad5)
- removed copper zone on B.Cu, net Net-(J1-Pad6)
- removed copper zone on B.Cu, net Net-(J1-Pad7)
- removed copper zone on B.Cu, net Net-(J1-Pad8)
- removed copper zone on F.Cu, net Net-(J2-Pad1)
- removed copper zone on F.Cu, net Net-(J2-Pad2)
- removed copper zone on F.Cu, net Net-(J2-Pad3)
- removed copper zone on F.Cu, net Net-(J2-Pad4)
- removed copper zone on F.Cu, net Net-(J2-Pad5)
- removed copper zone on F.Cu, net Net-(J2-Pad6)
- removed copper zone on F.Cu, net Net-(J2-Pad7)
- removed copper zone on F.Cu, net Net-(J2-Pad8)
Other:
- board text added: "1"
- board text added: "2"
- board text added: "3"
- board text added: "4"
- board text added: "5"
- board text added: "6"
- board text added: "7"
- board text added: "8"
- board text added: "Ruuvi"
