File: connector-breakout-a1/connector-breakout-a1.sch (KiCad schematic (older format))
At the start: 10 parts, among them J1 Ruuvi Connector Horizontal, J2 Ruuvi Connector Pin Header, J3 Ruuvi Connector Pin Header, J4 Ruuvi Connector Horizontal

Commit message: First draft
Parts:
- removed J1: Ruuvi Connector Horizontal, connector:RUUVI_CONNECTOR_FFC, symbol Connector_Generic:Conn_01x08
- added C1: 100n, passives:CAPC160X80X35L25N, symbol Device:C
- added JP1, JP2, JP3: SolderJumper_3_Open, Jumper:SolderJumper-3_P2.0mm_Open_TrianglePad1.0x1.5mm_NumberLabels, symbol Jumper:SolderJumper_3_Open
- added R1, R2: 10k, passives:CAPC160X80X35L25N, symbol Device:R
- added U1: NPA-700, Package_SO:SOIC-14W_7.5x9mm_P1.27mm, symbol npa-700:NPA-700
Connections:
- net VDD: now reaches J3.1 (Pin_1)
- net VDD: now also J2.1 (Pin_1), J4.1 (Pin_1), C1.2, JP1.3 (B), JP2.3 (B), JP3.3 (B), R1.1, R2.1, U1.7 (VDD)
- net SCL: now reaches J3.2 (Pin_2)
- net SCL: now also J2.2 (Pin_2), J4.2 (Pin_2), R1.2, U1.9 (SCL)
- net SDA: now reaches J3.3 (Pin_3)
- net SDA: now also J2.3 (Pin_3), J4.3 (Pin_3), R2.2, U1.8 (SDA)
- net GPIO3: now reaches J3.4 (Pin_4)
- net GPIO3: now also J2.4 (Pin_4), J4.4 (Pin_4), JP1.2 (C)
- net GPIO4: now reaches J3.5 (Pin_5)
- net GPIO4: now also J2.5 (Pin_5), J4.5 (Pin_5), JP2.2 (C)
- net GPIO5: now reaches J3.6 (Pin_6)
- net GPIO5: now also J2.6 (Pin_6), J4.6 (Pin_6), JP3.2 (C)
- net GPIO6: now reaches J3.7 (Pin_7)
- net GPIO6: now also J2.7 (Pin_7), J4.7 (Pin_7)
- net GND: now reaches J3.8 (Pin_8)
- net GND: now also J2.8 (Pin_8), J4.8 (Pin_8), C1.1, JP1.1 (A), JP2.1 (A), JP3.1 (A), U1.6 (VSS)
Other:
- note added: "GPIO3 | GPIO4 | GPIO5 | Sensor\n———————————————————————————\nHI | HI | LO/NC | \nLO/NC | HI | LO/NC|NPA-7xx-030D \nHI |LO/NC | LO/NC|NPA-7xx-015D\nLO/NC |LO/NC | LO/NC|NPA-7xx-005D\nHI | HI | LO/NC |NPA-7xx-001D\nLO/NC | HI | LO/NC |NPA-7xx-10WD\nHI |LO/NC | LO/NC |NPA-7xx-05WD\nLO/NC |LO/NC | LO/NC|NPA-7xx-02WD"
- note removed: "Bottom"
- moved on the sheet: H1, H2, H3, H4, H5, H6, J4
